File: BluePill.sch (EAGLE design)
At the start: 42 parts, among them X1 MST2V

Commit message: Add files via upload
Parts:
- removed G: (no value), adafruit:PINHD-1X3
- removed GND, SINAL: (no value), pinhead:PINHD-1X16
- removed USB: PN61729-S, con-berg:PN61729-S
- added D1: schottky, diode:DIODE-DO-214AC
- added GND2, SAIDAS: (no value), pinhead:PINHD-1X5
- added JP1: (no value), pinhead:PINHD-2X5
- added JP2: (no value), Seeed-Connector:DIP-USB-B-TYPE-FMAL(4+2P-2.0-90D)
- added JP3, JP4, JP5: (no value), pinhead:PINHD-1X7
- added JP6, JP7, USB_EXT: (no value), pinhead:PINHD-1X4
- added X2, X3, X4, X5: 1751264, con-phoenix-350:1751264
- 5V: device adafruit:PINHD-1X3 -> pinhead:PINHD-1X5
Connections:
- new net USB5V: D1.A, JP2.VBUS, USB_EXT.1
- net 1A_X: now also X2-4.K
- net 1B_X: now also X2-3.K
- net 2A_X: now also X2-2.K
- net 2B_X: now also X2-1.K
- net 3V3: no longer MSA.2, MSA.4, MSA.6, MSX.2, MSX.4, MSX.6, MSY.2, MSY.4, MSY.6, MSZ.2, MSZ.4, MSZ.6
- net 5V: now also 5V.4, 5V.5, D1.C, JP1.1, JP1.3, JP1.5, JP1.7, JP1.9, JP3.1, JP3.2, JP3.3, JP3.4, JP3.5, JP3.6, JP3.7, MSA.2, MSA.4, MSA.6, MSX.2, MSX.4, MSX.6, MSY.2, MSY.4, MSY.6, MSZ.2, MSZ.4, MSZ.6; no longer USB.1
- net COOL_FLOOD: now also SAIDAS.4; no longer SINAL.1
- net COOL_MIST: now also SAIDAS.5; no longer SINAL.2
- net CTL_CYCLESTART: now also JP6.3; no longer SINAL.3
- net CTL_FEEDHOLD: now also JP6.2; no longer SINAL.4
- net CTL_RESET: now also JP6.1; no longer SINAL.5
- net CTL_SAFETYDOOR: now also JP6.4; no longer SINAL.6
- net GND: now also GND2.1, GND2.2, GND2.3, GND2.4, GND2.5, JP1.10, JP1.2, JP1.4, JP1.6, JP1.8, JP2.GND, JP4.1, JP4.2, JP4.3, JP4.4, JP4.5, JP4.6, JP4.7, JP7.1, JP7.2, JP7.3, JP7.4, USB_EXT.4; no longer G.1, G.2, G.3, GND.1, GND.10, GND.11, GND.12, GND.13, GND.14, GND.15, GND.16, GND.2, GND.3, GND.4, GND.5, GND.6, GND.7, GND.8, GND.9, USB.4
- net N$21: now also X3-1.K
- net N$22: now also X3-2.K
- net N$23: now also X3-3.K
- net N$24: now also X3-4.K
- net N$25: now also X4-1.K
- net N$26: now also X4-2.K
- net N$27: now also X4-3.K
- net N$28: now also X4-4.K
- net N$29: now also X5-1.K
- net N$30: now also X5-2.K
- net N$31: now also X5-3.K
- net N$32: now also X5-4.K
- net SPINDLE_DIR: now also SAIDAS.2; no longer SINAL.7
- net SPINDLE_ENABLE: now also SAIDAS.1; no longer SINAL.8
- net SPINDLE_PWM: now also SAIDAS.3; no longer SINAL.9
- net USB_DM: now also JP2.D-, USB_EXT.2; no longer USB.2
- net USB_DP: now also JP2.D+, USB_EXT.3; no longer USB.3
- net XLIMIT: now also JP5.1, JP5.2; no longer SINAL.10, SINAL.11
- net YLIMIT: now also JP5.3, JP5.4; no longer SINAL.12, SINAL.13
- net ZLIMIT: now also JP5.5, JP5.6; no longer SINAL.14, SINAL.15
- net Z_PROBE: now also JP5.7; no longer SINAL.16
Other:
- note added: "!!!"
- note added: "5v"
